Commit message: Abel_Move final pkgs

File: abel_move/scripts/abel_arms_full.urdf (robot description, URDF)
Before this commit: robot abel_left_arm, 13 links, 12 joints
Links:
- link link_D10_EE: geometry collision cylinder length=0.35 radius=0.04; visual cylinder length=0.35 radius=0.03
- link link_D11_D12: geometry collision cylinder length=0.1 radius=0.04; visual cylinder length=0.1 radius=0.04
- link link_D12_D13: geometry collision cylinder length=0.09 radius=0.04; visual cylinder length=0.09 radius=0.04
- link link_D13_D14: geometry collision cylinder length=0.2 radius=0.04; visual cylinder length=0.2 radius=0.04
- link link_D14_D15: geometry collision cylinder length=0.08 radius=0.03; visual cylinder length=0.08 radius=0.03
- link link_D15_EE: geometry collision cylinder length=0.35 radius=0.04; visual cylinder length=0.35 radius=0.03
- link link_D6_D7: geometry collision cylinder length=0.1 radius=0.04; visual cylinder length=0.1 radius=0.04
- link link_D7_D8: geometry collision cylinder length=0.09 radius=0.04; visual cylinder length=0.09 radius=0.04
- link link_D8_D9: geometry collision cylinder length=0.2 radius=0.04; visual cylinder length=0.2 radius=0.04
- link link_D9_D10: geometry collision cylinder length=0.08 radius=0.03; visual cylinder length=0.08 radius=0.03
- link link_EE_L: geometry collision cylinder length=0.06 radius=0.04; visual cylinder length=0.06 radius=0.04
- link link_EE_R: geometry collision cylinder length=0.06 radius=0.04; visual cylinder length=0.06 radius=0.04
Joints:
- joint joint_D11: limit lower=-0.26 upper=3.14 effort=300 velocity=10 -> lower=-3.14 upper=0.261799 effort=300 velocity=10
- joint joint_D12: limit lower=-0.0872665 upper=1.55 effort=300 velocity=10 -> lower=-0.0872665 upper=2.96706 effort=300 velocity=10
- joint joint_D13: limit lower=-1 upper=1.25 effort=300 velocity=10 -> lower=-2.18166 upper=0.610865 effort=300 velocity=10
- joint joint_D14: limit lower=-2.26893 upper=0 effort=300 velocity=10 -> lower=0 upper=2.26893 effort=300 velocity=10
- joint joint_D7: limit lower=-0.0872665 upper=1.55 effort=300 velocity=10 -> lower=-0.0872665 upper=2.96706 effort=300 velocity=10
- joint joint_D8: limit lower=-1.25 upper=1 effort=300 velocity=10 -> lower=-2.18166 upper=0.610865 effort=300 velocity=10

Commit message: MoveIt integration and general fixes

File: abel_move/scripts/abel_arms_full.urdf (robot description, URDF)
Before this commit: robot abel_left_arm, 13 links, 12 joints
Links:
- removed link link_EE_L
- removed link link_EE_R
- link link_D10_EE: geometry collision cylinder length=0.32 radius=0.02; visual cylinder length=0.32 radius=0.02
- link link_D11_D12: geometry collision cylinder length=0.15 radius=0.02; visual cylinder length=0.15 radius=0.02
- link link_D12_D13: geometry collision cylinder length=0.04 radius=0.02; visual cylinder length=0.04 radius=0.02
- link link_D13_D14: geometry collision cylinder length=0.23 radius=0.02; visual cylinder length=0.23 radius=0.02
- link link_D14_D15: geometry collision cylinder length=0.04 radius=0.02; visual cylinder length=0.04 radius=0.02
- link link_D15_EE: geometry collision cylinder length=0.32 radius=0.02; visual cylinder length=0.32 radius=0.02
- link link_D6_D7: geometry collision cylinder length=0.15 radius=0.02; visual cylinder length=0.15 radius=0.02
- link link_D7_D8: geometry collision cylinder length=0.04 radius=0.02; visual cylinder length=0.04 radius=0.02
- link link_D8_D9: geometry collision cylinder length=0.23 radius=0.02; visual cylinder length=0.23 radius=0.02
- link link_D9_D10: geometry collision cylinder length=0.04 radius=0.02; visual cylinder length=0.04 radius=0.02
Joints:
- removed joint joint_EE
- removed joint joint_EE_L
- joint joint_D10: limit lower=-1.48353 upper=0.523599 effort=300 velocity=10 -> lower=-0.93 upper=1.08 effort=300 velocity=80; origin xyz=-0.065 0 0 rpy=3.14 -1.57 0 -> xyz=-0.065 -0.035 0 rpy=3.14 -1.57 0.5
- joint joint_D11: axis 0 0 1 -> 0 0 -1; limit lower=-3.14 upper=0.261799 effort=300 velocity=10 -> lower=-1.5 upper=0.2 effort=300 velocity=80
- joint joint_D12: axis 0 0 1 -> 0 0 -1; limit lower=-0.0872665 upper=2.96706 effort=300 velocity=10 -> lower=-1.2 upper=0.3 effort=300 velocity=80; origin xyz=0 0 0.08 rpy=-1.57 -1.57 0 -> xyz=0 0 0.08 rpy=-1.57 -1.3 0.25
- joint joint_D13: limit lower=-2.18166 upper=0.610865 effort=300 velocity=10 -> lower=-0.87 upper=1.5 effort=300 velocity=80
- joint joint_D14: axis 0 0 1 -> 0 0 -1; limit lower=0 upper=2.26893 effort=300 velocity=10 -> lower=-1 upper=1 effort=300 velocity=80; origin xyz=0 0 -0.125 rpy=0 -1.57 0 -> xyz=0 0 -0.125 rpy=0.5 -1.57 0
- joint joint_D15: limit lower=-1.48353 upper=0.523599 effort=300 velocity=10 -> lower=-1 upper=1 effort=300 velocity=80; origin xyz=-0.065 0 0 rpy=0 1.57 0 -> xyz=-0.065 0.035 0 rpy=0.5 1.57 0
- joint joint_D6: axis 0 0 1 -> 0 0 -1; limit lower=-3.14 upper=0.261799 effort=300 velocity=10 -> lower=-0.2 upper=1.5 effort=300 velocity=80
- joint joint_D7: limit lower=-0.0872665 upper=2.96706 effort=300 velocity=10 -> lower=-0.04 upper=1.5 effort=300 velocity=80; origin xyz=0 0 0.08 rpy=-1.57 -1.57 0 -> xyz=0 0 0.08 rpy=-1.57 -1.3 -0.25
- joint joint_D8: limit lower=-2.18166 upper=0.610865 effort=300 velocity=10 -> lower=-2 upper=0.94 effort=300 velocity=80
- joint joint_D9: axis 0 0 1 -> 0 0 -1; limit lower=0 upper=2.26893 effort=300 velocity=10 -> lower=-1.2 upper=0.2 effort=300 velocity=80; origin xyz=0 0 -0.125 rpy=0 -1.57 3.14 -> xyz=0 0 -0.125 rpy=-0.5 -1.57 3.14
