Commit message: General update with new packages

File: abel_description/urdf/abel_arms_full.urdf (robot description, URDF)
Before this commit: robot abel, 11 links, 10 joints
Links:
- added link link_EE_L; collision cylinder length=0.04 radius=0.02; visual cylinder length=0.04 radius=0.02
- added link link_EE_R; collision cylinder length=0.04 radius=0.02; visual cylinder length=0.04 radius=0.02
- link link_D10_EE: geometry collision cylinder length=0.35 radius=0.02; visual cylinder length=0.35 radius=0.02
- link link_D11_D12: geometry visual cylinder length=0.05 radius=0.02
- link link_D13_D14: geometry collision cylinder length=0.1 radius=0.02; visual cylinder length=0.1 radius=0.02
- link link_D15_EE: geometry collision cylinder length=0.35 radius=0.02; visual cylinder length=0.35 radius=0.02
- link link_D6_D7: geometry visual cylinder length=0.05 radius=0.02
- link link_D8_D9: geometry collision cylinder length=0.1 radius=0.02; visual cylinder length=0.1 radius=0.02
Joints:
- added joint joint_EE_L: type fixed, parent link_D10_EE, child link_EE_L, origin xyz=0 0 -0.40 rpy=0 1.57 0, axis 0 0 1, limit lower=-0.25 upper=0.25 effort=300 velocity=80
- added joint joint_EE_R: type fixed, parent link_D15_EE, child link_EE_R, origin xyz=0 0 -0.40 rpy=0 1.57 0, axis 0 0 1, limit lower=-0.25 upper=0.25 effort=300 velocity=80
- joint joint_D10: origin xyz=-0.065 -0.035 0 rpy=3.14 -1.57 0.5 -> xyz=-0.065 -0.065 0 rpy=3.14 -1.57 1
- joint joint_D11: origin xyz=0.10 0 0 rpy=0 -1.57 3.14 -> xyz=0.07 0 0 rpy=0 -1.57 3.14
- joint joint_D12: origin xyz=0 0 0.08 rpy=-1.57 -1.3 0.25 -> xyz=0 0 0.08 rpy=-1.57 -1.309 0.25
- joint joint_D13: origin xyz=0 -0.095 0 rpy=-1.57 0 0 -> xyz=0 -0.10 0 rpy=-1.57 0 0
- joint joint_D14: limit lower=-1 upper=1 effort=300 velocity=80 -> lower=-0.7 upper=0.8 effort=300 velocity=80; origin xyz=0 0 -0.125 rpy=0.5 -1.57 0 -> xyz=0 0 -0.13 rpy=0 -1.57 0
- joint joint_D15: origin xyz=-0.065 0.035 0 rpy=0.5 1.57 0 -> xyz=-0.065 0.065 0 rpy=1 1.57 0
- joint joint_D6: origin xyz=-0.10 0 0 rpy=0 -1.57 0 -> xyz=-0.07 0 0 rpy=0 -1.57 0
- joint joint_D7: limit lower=-0.04 upper=1.5 effort=300 velocity=80 -> lower=-0.04 upper=1.7 effort=300 velocity=80; origin xyz=0 0 0.08 rpy=-1.57 -1.3 -0.25 -> xyz=0 0 0.08 rpy=-1.57 -1.309 -0.25
- joint joint_D8: origin xyz=0 -0.095 0 rpy=-1.57 3.14 0 -> xyz=0 -0.10 0 rpy=-1.57 3.14 0
- joint joint_D9: limit lower=-1.2 upper=0.2 effort=300 velocity=80 -> lower=-0.8 upper=0.7 effort=300 velocity=80; origin xyz=0 0 -0.125 rpy=-0.5 -1.57 3.14 -> xyz=0 0 -0.13 rpy=0 -1.57 3.14
